File: ETAG_v10.3_NOSDTRANS.brd (EAGLE design)
At the start: 68.6 x 53.3 mm, 82 parts, among them Q1 FDN360P, Y4 32,768Khz

Commit message: updated hardware files
Finally put the new board file up. (v10.3)
Parts:
- removed BAT: 10MM_SM_COIN_CELL_CLIP, battery:10MM_SM_COIN_CELL_CLIP
- removed CR2A, CR2B: 100pF, rcl:C0603-ROUND
- removed FD1, FD2, FD3: FIDUCIALMOUNT, SmartPrj:FIDUCIA-MOUNT
- removed JPA, JPB: NA, pinhead:1X02
- removed SDPD, SDPU: 10k, Resistenze:R0603-ROUND
- removed T_SD: P_CHANNEL_MOSFET_, transistor-fet:SOT23
- added 3V, CK, GD, IO, RE: TPTP12R, testpad:TP12R
- added ANT: (no value), pinhead:1X04
- added U$1: 16M_COIN_SMTTHROUGH_HOLE, battery:16_MM_THROUGH_HOLE
- added U$2, U$3, U$4: (no value), fiducial:SQUARE-1MM-3R
- added UNA, UNB: (no value), rcl:C0603-ROUND
- AT_SAM: value SAMD21J18A -> SAMD
- CE1, CE2, CE3: device rcl:E2-5 -> rcl:PANASONIC_C
- moved RC 19.5 mm to (32.0, 31.3), turned to 0 degrees
- moved RD 19.4 mm to (32.0, 32.9), turned to 0 degrees
- moved CE1 17.0 mm to (23.1, 29.2), turned to 180 degrees
- moved CE2 16.9 mm to (15.0, 29.2), turned to 180 degrees
- moved CREF 8.20 mm to (28.9, 45.4)
- moved CD1A 3.21 mm to (24.0, 46.8)
- moved CD1B 3.17 mm to (13.1, 44.6), turned to 270 degrees
- moved CFA 3.15 mm to (26.1, 44.5)
- moved RFA 2.85 mm to (21.2, 40.4)
- moved CBLKA 2.76 mm to (21.9, 34.0)
- moved CGB 2.69 mm to (13.1, 38.4)
- moved CV2A 2.68 mm to (18.8, 34.0)
- moved CV1A 2.65 mm to (15.7, 34.0)
- moved L6 2.51 mm to (52.8, 12.2)
- moved RFB 2.46 mm to (8.03, 39.9)
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Connections:
- removed net N$14: CR1A.2, CR2A.2, CV1A.1, JPA.1
- removed net N$22: JPB.2, RAB.1
- removed net N$35: JPA.2, RAA.1
- removed net VDD: SD.4, T_SD.3
- new net AANT: ANT.4, RAA.1
- new net BANT: ANT.2, RAB.1
- new net CVA: ANT.3, CR1A.2, CV1A.1, UNA.2
- net +3V3: now also 3V.TP, SD.4; no longer SDPU.2, T_SD.2
- net CVB: now also ANT.1, UNB.2; no longer CR2B.2, JPB.1
- net GND: now also GD.TP, U$1.P$3; no longer BAT.-, SDPD.1
- net N$12: now also UNA.1; no longer CR2A.1
- net N$23: now also U$1.P$1; no longer BAT.+@1, BAT.+@2
- net N$7: now also UNB.1; no longer CR2B.1
- net RESET: now also RE.TP
- net SD_FET: no longer SDPD.2, SDPU.1, T_SD.1
- net SWCLK: now also CK.TP
- net SWDIO: now also IO.TP
Routing:
- net SD_FET: track 31.9 -> 0.00 mm, vias 2 -> 0
- net +3V3: track 220.7 -> 246.8 mm, vias 11 -> 13
- net N$14: track 21.7 -> 0.00 mm, vias 1 -> 0
- net CVA: track 0.00 -> 18.8 mm, vias 0 -> 1
- net GND: track 51.0 -> 66.7 mm, vias 51 -> 61
- net SPI_MISO: track 58.6 -> 73.4 mm, vias 2 -> 1
- net N$35: track 10.8 -> 0.00 mm, vias 1 -> 0
- net I2C_SDA: track 50.6 -> 40.9 mm
- net V_IN: track 189.8 -> 180.4 mm, vias 7 -> 4
- net SPI_MOSI: track 52.6 -> 61.8 mm
- net N$22: track 8.99 -> 0.00 mm
- net SWDIO: track 24.5 -> 32.9 mm
- net AANT: track 0.00 -> 8.07 mm
- net BANT: track 0.00 -> 7.78 mm
- net SWCLK: track 29.2 -> 34.8 mm
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Other:
- board text added: "21J"
- board text added: "<-ON BATTERY | ON USB->"
- board text added: "RFID Arduino V10.1 Eli Bridge - Univ of Okla Jay Wilhelm - Ohio Univ January 2023"
- board text removed: "<-ON BATTERY"
- board text removed: "ON USB->"
- board text removed: "Pin 1"
- board text removed: "RFID Arduino Eli Bridge - University of Oklahoma Jay Wilhelm - Ohio University July 2019"
