File: ETAG_v10.3_NOSDTRANS.sch (EAGLE design)
At the start: 82 parts, among them Q1 FDN360P, Y4 32,768Khz

Commit message: updated hardware files
Finally put the new board file up. (v10.3)
Parts:
- removed BAT: 10MM_SM_COIN_CELL_CLIP, battery:10MM_SM_COIN_CELL_CLIP
- removed FD1, FD2, FD3: FIDUCIALMOUNT, SmartPrj:FIDUCIALMOUNT
- removed JPA, JPB: NA, pinhead:PINHD-1X2
- removed SDPD, SDPU: 10k, Resistenze:0028_CR0603JW103L
- removed T_SD: P_CHANNEL_MOSFET_, transistor-fet:P_CHANNEL_MOSFET_
- added 3V, CK, GD, IO, RE: TPTP12R, testpad:TPTP12R
- added ANT: (no value), pinhead:PINHD-1X4
- added U$1: 16M_COIN_SMTTHROUGH_HOLE, battery:16M_COIN_SMTTHROUGH_HOLE
- AT_SAM: value SAMD21J18A -> SAMD
- CE1, CE2, CE3: device rcl:CPOL-USE2-5 -> rcl:CPOL-USC
- UNA, UNB: value 100pF -> (none)
- renumbered CR2A to UNA, CR2B to UNB
Connections:
- removed net N$14: CR1A.2, CV1A.1, JPA.1, UNA.2
- removed net N$22: JPB.2, RAB.1
- removed net N$35: JPA.2, RAA.1
- removed net VDD: SD.VDD, T_SD.D
- new net AANT: ANT.4, RAA.1
- new net BANT: ANT.2, RAB.1
- new net CVA: ANT.3, CR1A.2, CV1A.1, UNA.2
- net +3V3: now also 3V.TP, SD.VDD; no longer SDPU.2, T_SD.S
- net CVB: now also ANT.1; no longer JPB.1
- net GND: now also GD.TP, U$1.-; no longer BAT.-, SDPD.1
- net N$23: now also U$1.+; no longer BAT.+
- net RESET: now also RE.TP
- net SD_FET: no longer SDPD.2, SDPU.1, T_SD.G
- net SWCLK: now also CK.TP
- net SWDIO: now also IO.TP
